File: schematic.kicad_sch (KiCad schematic)
At the start: 8 parts, among them J1 output, J2 output

Commit message: shematic updatet
Parts:
- added J3: scope CH2 (Y), symbol Connector:Conn_01x01_Pin
- added J4: ADC tap GP27 (Y), symbol Connector:Conn_01x01_Pin
- added J5: Ch1 Ground, symbol Connector:Conn_01x01_Pin
- added J6: Ch2 Ground, symbol Connector:Conn_01x01_Pin
- J1: value output -> scope CH1 (X)
- J2: value output -> ADC tap GP26 (X)
Connections:
- net GND: now also V2.1, J5.1 (Pin_1), J6.1 (Pin_1); no longer V2.2
- net at C1.1, J1.1 (Pin_1), R2.1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: now also J2.1 (Pin_1)
- net at R1.2: now also C2.1, J3.1 (Pin_1), J4.1 (Pin_1); no longer V2.1
- new net: R1.1, V2.2
Other:
- moved on the sheet: C1, C2, J1, J2, R1, R2, V1, V2
